File: PCB/aegis/_autosave-aegis.kicad_pcb (KiCad board)
At the start: 2 copper layers, 323.8 x 169.8 mm, 108 parts, among them Q1 TIP120, U1 ProMicro

Commit message: save
Other:
- board outline removed
