File: PCB/aegis/aegis.kicad_pcb (KiCad board)
At the start: 2 copper layers, 323.8 x 169.8 mm, 108 parts, among them Q1 TIP120, U1 ProMicro

Commit message: update
Parts:
- removed the D2 at (-16.2, 321.9)
- added G***: LOGO, cc:cc, F.Cu at (187.2, 134.4)
- LED1, LED10, LED11, LED12, LED13, LED14, LED15, LED2, LED3, LED4, LED5, LED6, LED7, LED9: moved to F.Cu
- LED8, R1: moved to B.Cu
- Solenoide1: footprint Connector_PinHeader_1.00mm:PinHeader_1x02_P1.00mm_Vertical -> Connector_PinHeader_1.27mm:PinHeader_1x02_P1.27mm_Horizontal
- moved MX3 288.4 mm to (-5.88, 54.1), turned to 328 degrees
- moved MX2 286.5 mm to (4.13, 38.0), turned to 328 degrees
- moved MX1 284.8 mm to (14.2, 21.9), turned to 328 degrees
- moved D3 283.2 mm to (2.63, 58.3), turned to 58 degrees
- moved LED4 282.3 mm to (7.14, 51.0), turned to 328 degrees
- moved D2 281.2 mm to (12.7, 42.1), turned to 58 degrees
- moved LED3 280.4 mm to (17.3, 34.7), turned to 148 degrees
- moved D1 279.5 mm to (22.9, 25.8), turned to 58 degrees
- moved MX6 278.2 mm to (10.2, 64.2), turned to 328 degrees
- moved MX5 276.1 mm to (20.3, 48.1), turned to 328 degrees
- moved MX4 274.4 mm to (30.3, 31.9), turned to 328 degrees
- moved D6 273.0 mm to (18.9, 68.1), turned to 58 degrees
- moved D5 270.9 mm to (29.0, 52.0), turned to 58 degrees
- moved D4 269.2 mm to (39.0, 35.9), turned to 58 degrees
- moved MX9 267.4 mm to (28.8, 70.2), turned to 328 degrees
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Routing:
- net VCC: track 782.0 -> 695.8 mm, vias 14 -> 17
- net GND: track 792.2 -> 783.5 mm, vias 16 -> 17
- net Net-(LED3-Pad2): track 31.9 -> 24.1 mm
- net Net-(LED11-Pad2): track 62.8 -> 56.1 mm, vias 2 -> 0
- net ROW5: track 423.7 -> 427.5 mm
- net RAW: track 91.0 -> 94.6 mm
- net Net-(LED12-Pad2): track 22.0 -> 24.1 mm
- net ROW1: track 465.3 -> 467.4 mm
- net Net-(LED6-Pad2): track 35.7 -> 37.6 mm, vias 2 -> 0
- net Net-(LED7-Pad2): track 29.3 -> 31.2 mm
- net Net-(LED4-Pad2): track 55.7 -> 57.3 mm, vias 2 -> 0
- net Net-(LED14-Pad2): track 33.9 -> 35.4 mm, vias 0 -> 2
- net LED: track 113.3 -> 114.8 mm, vias 2 -> 1
- net Net-(LED10-Pad4): track 26.7 -> 25.3 mm
- net Net-(Diode1-Pad2): track 39.9 -> 41.3 mm
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Other:
- outline, holes or cut-outs redrawn
- board text added: "Aegis v1. u/Coumbaya"
- board text added: "Solenoid"
- board text added: "USB UP"
- board text added: "inverted"

Commit message: update PCB to v1.1
Parts:
- added RAW -> SOL: Jumper_NO_Small, Jumper:SolderJumper-2_P1.3mm_Open_Pad1.0x1.5mm, B.Cu at (149.0, 96.7)
- added VCC -> SOL: Jumper_NO_Small, Jumper:SolderJumper-2_P1.3mm_Open_Pad1.0x1.5mm, B.Cu at (151.0, 102.1)
- Solenoide1: footprint Connector_PinHeader_1.27mm:PinHeader_1x02_P1.27mm_Horizontal -> footprints:ResetSW
- moved MX32 14.1 mm to (264.2, 126.9)
- moved MX25 14.1 mm to (226.2, 100.7)
- moved D32 14.1 mm to (273.7, 126.0)
- moved MX7 14.1 mm to (35.8, 43.0)
- moved D39 14.1 mm to (70.5, 129.9)
- moved D7 14.1 mm to (44.4, 47.0)
- moved D23 14.1 mm to (216.7, 121.2)
- moved D5 14.1 mm to (15.8, 57.0)
- moved D10 14.1 mm to (61.8, 55.1)
- moved LED12 14.1 mm to (273.6, 135.5)
- moved MX26 14.1 mm to (226.2, 119.7)
- moved MX6 14.1 mm to (-3.02, 69.2)
- moved LED13 14.1 mm to (273.8, 116.0)
- moved D27 14.1 mm to (235.7, 137.7)
- moved D14 14.1 mm to (66.3, 83.6)
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- renumbered OLED1 to OLED
Connections:
- Diode1 pad 1: RAW -> Net-(Diode1-Pad1)
- Solenoide1 pad 1: RAW -> Net-(Diode1-Pad1)
Routing:
- net Net-(Diode1-Pad1): track 0.00 -> 79.6 mm, vias 0 -> 3
- net RAW: track 94.6 -> 23.8 mm, vias 2 -> 1
- net VCC: track 695.8 -> 710.1 mm, vias 17 -> 18
- net Net-(Diode1-Pad2): track 41.3 -> 36.1 mm
- net Net-(LED7-Pad2): track 31.2 -> 30.5 mm
Other:
- outline, holes or cut-outs redrawn
- board text added: "Aegis v1.1 u/Coumbaya"
- board text removed: "Aegis v1. u/Coumbaya"
- board text removed: "Solenoid"
